File: _autosave-interfejs_digi.kicad_pcb (KiCad board)
At the start: 2 copper layers, 87.5 x 53 mm, 96 parts, among them J1 USB, J10 PTT, J11 FSK, J2 CI-V, J7 CAT_1, J8 CAT_2, J9 CW, Q1 2N7002, Q2 2N7002, Q3 2N7002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

Commit message: poprawki
Parts:
- moved G*** 27.2 mm to (88.0, 170.7)
Other:
- board text added: "github.com/ canislupus11/ Digi_interface"
