File: interfejs_digi.kicad_pcb (KiCad board)
At the start: 2 copper layers, 87.5 x 53 mm, 96 parts, among them J1 USB, J10 PTT, J11 FSK, J2 CI-V, J7 CAT_1, J8 CAT_2, J9 CW, Q1 2N7002, Q2 2N7002, Q3 2N7002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

Commit message: update
Other:
- rule pad_to_mask_clearance: 0.1 -> 0
Changed lines of the file:
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@@
 				(type "Bottom Silk Screen")
 			)
-			(copper_finish "HAL SnPb")
+			(copper_finish "ENIG")
 			(dielectric_constraints no)
 		)
-		(pad_to_mask_clearance 0.1)
+		(pad_to_mask_clearance 0)
 		(allow_soldermask_bridges_in_footprints no)
 		(tenting front back)
