File: interfejs_digi.kicad_pcb (KiCad board)
At the start: 2 copper layers, 87.5 x 53 mm, 96 parts, among them J1 USB, J10 PTT, J11 FSK, J2 CI-V, J7 CAT_1, J8 CAT_2, J9 CW, Q1 2N7002, Q2 2N7002, Q3 2N7002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

Commit message: update
Parts:
- moved G*** 0.11 mm to (88.0, 170.6)

Commit message: update
Other:
- board text added: "AUDIO_IN AUDIO_OUT GND PTT_OUT PWR_IN GND_IN CAT_1_TX CAT_1_RX"
- board text removed: "AUDIO_IN AUDIO_OUT GND PTT_OUT 12V_IN GND_IN CAT_1_TX CAT_1_RX"
Changed lines of the file:
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@@
 		)
 	)
-	(gr_text "AUDIO_IN\nAUDIO_OUT\nGND\nPTT_OUT\n12V_IN\nGND_IN\nCAT_1_TX\nCAT_1_RX"
+	(gr_text "AUDIO_IN\nAUDIO_OUT\nGND\nPTT_OUT\nPWR_IN\nGND_IN\nCAT_1_TX\nCAT_1_RX"
 		(at 120.8 170.622824 270)
 		(layer "B.SilkS")

Commit message: update
Parts:
- added G***: LOGO, LOGO, F.Cu at (126.3, 84.3)
- moved C10 118.0 mm to (96.0, 56.0)
- moved C11 118.0 mm to (94.5, 56.0)
- moved C12 118.0 mm to (105.7, 59.3)
- moved C13 118.0 mm to (103.5, 56.0)
- moved C14 118.0 mm to (100.5, 56.0)
- moved C15 118.0 mm to (97.5, 56.0)
- moved C16 118.0 mm to (102.0, 56.0)
- moved C19 118.0 mm to (106.7, 79.6)
- moved C26 118.0 mm to (99.0, 56.0)
- moved C28 118.0 mm to (98.1, 81.1)
- moved C4 118.0 mm to (122.9, 79.8)
- moved C5 118.0 mm to (122.9, 76.8)
- moved C6 118.0 mm to (117.4, 82.4)
- moved C7 118.0 mm to (122.9, 73.8)
- moved D10 118.0 mm to (105.4, 71.5)
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Other:
- outline, holes or cut-outs redrawn
