File: interfejs_digi.kicad_sch (KiCad schematic)
At the start: 78 parts, among them J1 USB, J10 PTT, J11 FSK, J2 CI-V, J7 CAT_1, J8 CAT_2, J9 CW, Q1 2N7002, Q2 2N7002, Q3 2N7002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

Commit message: update
Other:
- company: (none) -> Hackerspace Cracow Foundation
- title: (none) -> Universal ham radio interface
- moved on the sheet: C1, C10, C11, C12, C13, C14, C15, C16, C17, C18, C19, C2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

Commit message: update
Parts:
- U1: value ADUM4160 -> ADUM3160; LCSC C57791 -> C284149
Changed lines of the file:
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@@
 			)
 		)
-		(property "Value" "ADUM4160"
+		(property "Value" "ADUM3160"
 			(at 158.3533 78.74 0)
 			(effects
@@
 			)
 		)
-		(property "LCSC" "C57791"
+		(property "LCSC" "C284149"
 			(at 153.67 92.71 0)
 			(effects

Commit message: update
Connections:
- net 12V_IN renamed PWR_IN
Changed lines of the file:
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@@
 		)
 	)
-	(global_label "12V_IN"
+	(global_label "PWR_IN"
 		(shape input)
 		(at 478.79 224.79 180)
@@
 		)
 		(property "Intersheetrefs" "${INTERSHEET_REFS}"
-			(at 470.0485 224.79 0)
+			(at 469.5647 224.79 0)
 			(effects
 				(font
@@
 		)
 	)
-	(global_label "12V_IN"
+	(global_label "PWR_IN"
 		(shape input)
 		(at 80.01 294.64 180)
@@
 		)
 		(property "Intersheetrefs" "${INTERSHEET_REFS}"
-			(at 71.2685 294.64 0)
-			(effects
-				(font
+			(at 70.7847 294.64 0)
+			(effects
+				(font
