File: KiCad/interfejs_digi.kicad_pcb (KiCad board)
At the start: 2 copper layers, 87.5 x 53 mm, 97 parts, among them J1 USB, J10 PTT, J11 FSK, J2 CI-V, J7 CAT_1, J8 CAT_2, J9 CW, Q1 2N7002, Q2 2N7002, Q3 2N7002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

Commit message: update
Other:
- board text added: "AUDIO_IN AUDIO_OUT GND PTT_OUT PWR_IN GND_IN CAT_1_TX CAT_1_RX (CI-V)"
- board text removed: "AUDIO_IN AUDIO_OUT GND PTT_OUT PWR_IN GND_IN CAT_1_TX CAT_1_RX"
Changed lines of the file:
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@@
 	)
 	(gr_line
-		(start 110.1625 44.247823)
+		(start 110.0125 44.197823)
 		(end 109.3625 47.447823)
 		(stroke
@@
 	)
 	(gr_line
-		(start 110.9625 46.047823)
-		(end 110.5625 47.647823)
+		(start 110.9625 45.897823)
+		(end 110.6125 47.497823)
 		(stroke
 			(width 0.15)
@@
 	)
 	(gr_line
-		(start 114.1625 44.447823)
-		(end 114.3625 48.047823)
+		(start 114.1625 44.247823)
+		(end 114.5125 47.997823)
 		(stroke
 			(width 0.15)
@@
 	(gr_line
 		(start 115.3625 46.047823)
-		(end 115.7125 50.247823)
-		(stroke
-			(width 0.15)
-			(type default)
-		)
-		(layer "B.SilkS")
-	)
-	(gr_line
-		(start 116.9625 46.647823)
-		(end 116.1625 44.447823)
+		(end 115.8125 50.497823)
+		(stroke
+			(width 0.15)
+			(type default)
+		)
+		(layer "B.SilkS")
+	)
+	(gr_line
+		(start 116.7625 46.647823)
+		(end 116.2125 44.197823)
 		(stroke
 			(width 0.15)
@@
 	(gr_line
 		(start 117.7625 45.847823)
-		(end 118.1625 46.647823)
+		(end 118.3125 47.547823)
 		(stroke
 			(width 0.15)
@@
 		)
 	)
-	(gr_text "AUDIO_IN\nAUDIO_OUT\nGND\nPTT_OUT\nPWR_IN\nGND_IN\nCAT_1_TX\nCAT_1_RX"
-		(at 108.7625 53.247823 270)
-		(layer "B.SilkS")
-		(effects
+	(gr_text "AUDIO_IN\nAUDIO_OUT\nGND\nPTT_OUT\nPWR_IN\nGND_IN\nCAT_1_TX\nCAT_1_RX\n(CI-V)"
+		(at 107.4625 53.297823 270)
+		(layer "B.SilkS")
+		(effects
