File: KiCad/interfejs_digi.kicad_pcb (KiCad board)
At the start: 2 copper layers, 87.5 x 53 mm, 97 parts, among them J1 USB, J10 PTT, J11 FSK, J2 CI-V, J7 CAT_1, J8 CAT_2, J9 CW, Q1 2N7002, Q2 2N7002, Q3 2N7002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

Commit message: update
Parts:
- added JP1: LDO_BYPASS, Jumper:SolderJumper-2_P1.3mm_Open_RoundedPad1.0x1.5mm, F.Cu at (129.4, 38.0)
- U1: value ADUM4160 -> ADUM3160
Connections:
- net 12V_IN renamed PWR_IN
Routing:
- net PWR_IN: track 25.2 -> 38.9 mm
- net +5V: track 196.6 -> 204.6 mm
- net GND: track 71.8 -> 65.9 mm, vias 590 -> 604
Other:
- board text added: "LDO BYPASS"
- board text added: "{ "ViaStitching": "0.2", "stitch_zone_0": { "HSpacing": "1.4", "VSpacing": "1.4", "HOffset": "0", "VOffset": "0", "Clearance": "0.2", "Randomize": false, "Stagger": true } }"
- board text added: "{ "ViaStitching": "0.2", "stitch_zone_0": { "HSpacing": "1.6", "VSpacing": "1.3", "HOffset": "0", "VOffset": "0", "Clearance": "0", "Randomize": false, "Stagger": true } }"
- board text added: "{ "ViaStitching": "0.2", "stitch_zone_0": { "HSpacing": "1.6", "VSpacing": "1.8", "HOffset": "0", "VOffset": "0", "Clearance": "0", "Randomize": false, "Stagger": true } }"
- board text added: "{ "ViaStitching": "0.2", "stitch_zone_0": { "HSpacing": "1.7", "VSpacing": "1.5", "HOffset": "0", "VOffset": "0", "Clearance": "0.2", "Randomize": false, "Stagger": true } }"

Commit message: update1
Other:
- board text added: "LDO_BYPASS"
- board text removed: "LDO BYPASS"
Changed lines of the file:
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@@
 		)
 	)
-	(gr_text "LDO BYPASS"
+	(gr_text "LDO_BYPASS"
 		(at 130.9625 38.597823 0)
 		(layer "F.SilkS")

Commit message: update
Connections:
- RJ2 pad 4: unconnected-(RJ2-Pad4) -> +5V
Routing:
- net RTS_2: track 89.6 -> 65.6 mm, vias 2 -> 4
- net RTS_1: track 79.4 -> 58.4 mm, vias 0 -> 2
- net +5V: track 204.6 -> 217.5 mm
- net FSK_OUT: track 72.1 -> 71.0 mm
- net GND: vias 604 -> 602
Other:
- board text added: "CW_OUT 5V_OUT FSK_OUT CAT_2_TX CAT_2_RX"
- board text removed: "CW_OUT FSK_OUT CAT_2_TX CAT_2_RX"

Commit message: zmiana wyjscia starujacego
Parts:
- added Q4: 2N7002, Package_TO_SOT_SMD:SOT-23, F.Cu at (145.2, 75.3)
- added Q5: 2N7002, Package_TO_SOT_SMD:SOT-23, F.Cu at (142.3, 63.7)
- added Q6: 2N7002, Package_TO_SOT_SMD:SOT-23, F.Cu at (142.2, 54.2)
- added R19: 22k, Resistor_SMD:R_0603_1608Metric, F.Cu at (145.8, 72.7)
- added R20: 22k, Resistor_SMD:R_0603_1608Metric, F.Cu at (145.8, 63.3)
- added R21: 22k, Resistor_SMD:R_0603_1608Metric, F.Cu at (145.8, 53.8)
- moved kibuzzard-69B08BB3 17.4 mm to (132.5, 84.9), turned to 0 degrees
- moved kibuzzard-69B08B92 16.2 mm to (132.7, 74.9), turned to 0 degrees
- moved kibuzzard-69B08B73 15.5 mm to (132.6, 64.9), turned to 0 degrees
- moved kibuzzard-69B08C88 9.99 mm to (139.4, 49.2)
- moved D6 6.46 mm to (142.4, 49.2), turned to 0 degrees
- moved R10 5.06 mm to (145.7, 49.2)
- moved D3 4.53 mm to (142.4, 59.0), turned to 0 degrees
- moved D2 3.73 mm to (142.5, 77.8), turned to 0 degrees
- moved D1 3.43 mm to (142.6, 68.4), turned to 0 degrees
- moved R8 3.39 mm to (145.8, 77.8), turned to 0 degrees
- moved R11 3.05 mm to (145.8, 59.0), turned to 0 degrees
- moved R7 2.69 mm to (145.9, 68.4), turned to 0 degrees
- moved Q3 2.44 mm to (145.2, 56.4), turned to 0 degrees
- moved Q1 2.22 mm to (145.3, 65.9), turned to 0 degrees
- moved kibuzzard-69B08B73 1.95 mm to (139.4, 58.9), turned to 90 degrees
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Connections:
- D1 pad 1: GND -> PTT
- D10 pad 1: Net-(D10-K) -> CAT1_TX_TTL
- D10 pad 2: CAT1_TX_TTL -> Net-(D10-A)
- D2 pad 1: GND -> FSK
- D3 pad 1: GND -> CW
- D6 pad 1: Net-(D6-K) -> GND
- D6 pad 2: +5V -> Net-(D6-A)
- D7 pad 1: Net-(D7-K) -> CAT2_RX_TTL
- D7 pad 2: CAT2_RX_TTL -> Net-(D7-A)
- D8 pad 1: Net-(D8-K) -> CAT1_RX_TTL
- D8 pad 2: CAT1_RX_TTL -> Net-(D8-A)
- D9 pad 1: Net-(D9-K) -> CAT2_TX_TTL
- D9 pad 2: CAT2_TX_TTL -> Net-(D9-A)
- Q1 pad 1: PTT -> Net-(Q1-G)
- Q2 pad 3: FSK_OUT -> Net-(Q2-D)
- Q3 pad 1: CW -> Net-(Q3-G)
- R10 pad 1: GND -> Net-(D6-A)
- R10 pad 2: Net-(D6-K) -> +5V
- R11 pad 2: CW -> +5V
- R12 pad 1: GND -> +5V
- R12 pad 2: Net-(D7-K) -> Net-(D7-A)
- R16 pad 1: GND -> +5V
- R16 pad 2: Net-(D8-K) -> Net-(D8-A)
- R17 pad 1: GND -> +5V
- R17 pad 2: Net-(D9-K) -> Net-(D9-A)
- R18 pad 1: GND -> +5V
- R18 pad 2: Net-(D10-K) -> Net-(D10-A)
- R7 pad 2: PTT -> +5V
- R8 pad 2: FSK -> +5V
- RJ1 pad 6: GND -> CW_OUT
Routing:
- net +5V: track 217.5 -> 244.8 mm, vias 88 -> 89
- net Net-(D7-K): track 18.3 -> 0.00 mm
- net Net-(D7-A): track 0.00 -> 18.3 mm
- net Net-(D9-K): track 15.4 -> 0.00 mm
- net Net-(D9-A): track 0.00 -> 15.4 mm
- net Net-(D10-K): track 15.0 -> 0.00 mm
- net Net-(D10-A): track 0.00 -> 15.0 mm
- net Net-(D8-K): track 14.3 -> 0.00 mm
- net Net-(D8-A): track 0.00 -> 14.3 mm
- net GND: track 65.9 -> 53.2 mm, vias 602 -> 594
- net CW_OUT: track 55.2 -> 66.8 mm, vias 2 -> 3
- net FSK_OUT: track 71.0 -> 78.4 mm
- net PTT_OUT: track 45.9 -> 52.0 mm
- net PTT: track 15.6 -> 19.8 mm
- net CW: track 15.8 -> 19.5 mm
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Other:
- board text added: "AUDIO_IN AUDIO_OUT CW_OUT PTT_OUT PWR_IN GND_IN CAT_1_TX CAT_1_RX (CI-V)"
- board text added: "DTR1 RTS1 RTS2"
- board text added: "DTR2 RTS2 RTS1"
- board text added: "{ "ViaStitching": "0.2", "stitch_zone_0": { "HSpacing": "1.7", "VSpacing": "1.5", "HOffset": "0", "VOffset": "0", "Clearance": "0.3", "Randomize": false, "Stagger": false } }"
- board text removed: "AUDIO_IN AUDIO_OUT GND PTT_OUT PWR_IN GND_IN CAT_1_TX CAT_1_RX (CI-V)"
- board text removed: "DTR1"
- board text removed: "DTR2"
- board text removed: "RTS1"
- board text removed: "RTS2"

Commit message: update
Parts:
- moved kibuzzard-69B08C88 0.30 mm to (139.4, 49.5)
- moved D6 0.30 mm to (142.4, 49.5)
- moved R10 0.30 mm to (145.7, 49.5)
- moved G*** 0.05 mm to (76.0, 53.2), turned to 90 degrees

Commit message: update
Routing:
- net GND: vias 594 -> 585

Commit message: update
Parts:
- moved D10 1.45 mm to (103.9, 71.5)
- moved D8 1.45 mm to (106.0, 71.5)
- moved kibuzzard-69E7E9BF 1.41 mm to (104.0, 75.7)
- moved kibuzzard-69E7EA0C 1.41 mm to (106.0, 75.7)
- moved kibuzzard-69E7EA01 0.15 mm to (109.6, 75.7)
- moved kibuzzard-69E7EA14 0.15 mm to (111.7, 75.7)
- moved D7 0.15 mm to (111.7, 71.5)
- moved D9 0.15 mm to (109.6, 71.5)
Routing:
- net CAT1_RX_TTL: track 68.1 -> 69.5 mm
- net CAT2_TX_TTL: track 41.8 -> 42.9 mm
- net CAT1_TX_TTL: track 73.3 -> 74.1 mm
- net Net-(D10-A): track 15.0 -> 15.8 mm
- net Net-(D7-A): track 18.3 -> 18.9 mm
- net GND: vias 585 -> 583
