File: KiCad/interfejs_digi.kicad_sch (KiCad schematic)
At the start: 78 parts, among them J1 USB, J10 PTT, J11 FSK, J2 CI-V, J7 CAT_1, J8 CAT_2, J9 CW, Q1 2N7002, Q2 2N7002, Q3 2N7002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

Commit message: update
Parts:
- added JP1: LDO_BYPASS, Jumper:SolderJumper-2_P1.3mm_Open_RoundedPad1.0x1.5mm, symbol Jumper:SolderJumper_2_Open
Connections:
- net +5V: now also JP1.2 (B)
- net PWR_IN: now also JP1.1 (A)
Changed lines of the file:
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@@
 	(wire
 		(pts
+			(xy 91.44 285.75) (xy 82.55 285.75)
+		)
+		(stroke
+			(width 0)
+			(type default)
+		)
+	)
+	(wire
+		(pts
 			(xy 82.55 304.8) (xy 95.25 304.8)
 		)
@@
 	(wire
 		(pts
+			(xy 82.55 285.75) (xy 82.55 294.64)
+		)
+		(stroke
+			(width 0)
+			(type default)
+		)
+	)
+	(wire
+		(pts
 			(xy 406.4 193.04) (xy 410.21 193.04)
 		)
@@
 	(wire
 		(pts
+			(xy 99.06 285.75) (xy 104.14 285.75)
+		)
+		(stroke
+			(width 0)
+			(type default)
+		)
+	)
+	(wire
+		(pts
 			(xy 151.13 113.03) (xy 151.13 107.95)
 		)
@@
 	(wire
 		(pts
+			(xy 104.14 285.75) (xy 104.14 294.64)
+		)
+		(stroke
+			(width 0)
+			(type default)
+		)
+	)
+	(wire
+		(pts
 			(xy 240.03 213.36) (xy 240.03 209.55)
 		)
@@
 					(unit 1)
 				)
+			)
+		)
+	)
+	(symbol
+		(lib_id "Jumper:SolderJumper_2_Open")
+		(at 95.25 285.75 0)
+		(unit 1)
+		(exclude_from_sim no)
+		(in_bom no)
+		(on_board yes)
+		(dnp no)
+		(fields_autoplaced yes)
+		(property "Reference" "JP1"
+			(at 95.25 279.4 0)
+			(effects
+				(font
+					(size 1.27 1.27)
+				)
+			)
+		)
+		(property "Value" "LDO_BYPASS"
+			(at 95.25 281.94 0)
+			(effects
+				(font
+					(size 1.27 1.27)
+				)
+			)
+		)
+		(property "Footprint" "Jumper:SolderJumper-2_P1.3mm_Open_RoundedPad1.0x1.5mm"
+			(at 95.25 285.75 0)
+			(effects
+				(font
+					(size 1.27 1.27)
+				)
+				(hide yes)
+			)
+		)
+		(property "Datasheet" "~"
+			(at 95.25 285.75 0)
+			(effects
+				(font
+					(size 1.27 1.27)
+				)
+				(hide yes)
+			)
+		)
+		(property "Description" "Solder Jumper, 2-pole, open"
+			(at 95.25 285.75 0)
+			(effects
+				(font
+					(size 1.27 1.27)
+				)
+				(hide yes)
+			)
+		)
+		(pin "2"
+		)
+		(pin "1"
+		)
+		(instances
+			(project "interfejs_digi"
+				(path "/7f52d787-caa3-4a92-b1b2-19d554dc29a4"
+					(reference "JP1")
+					(unit 1)
+				)

Commit message: update
Connections:
- net +5V: now also RJ2.4
Changed lines of the file:
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@@
 	(wire
 		(pts
+			(xy 469.9 251.46) (xy 478.79 251.46)
+		)
+		(stroke
+			(width 0)
+			(type default)
+		)
+	)
+	(wire
+		(pts
 			(xy 402.59 231.14) (xy 406.4 231.14)
 		)
@@
 					(unit 1)
 				)
+			)
+		)
+	)
+	(symbol
+		(lib_id "power:+5V")
+		(at 469.9 251.46 90)
+		(unit 1)
+		(exclude_from_sim no)
+		(in_bom yes)
+		(on_board yes)
+		(dnp no)
+		(property "Reference" "#PWR040"
+			(at 473.71 251.46 0)
+			(effects
+				(font
+					(size 1.27 1.27)
+				)
+				(hide yes)
+			)
+		)
+		(property "Value" "+5V"
+			(at 466.09 251.46 0)
+			(effects
+				(font
+					(size 1.27 1.27)
+				)
+			)
+		)
+		(property "Footprint" ""
+			(at 469.9 251.46 0)
+			(effects
+				(font
+					(size 1.27 1.27)
+				)
+				(hide yes)
+			)
+		)
+		(property "Datasheet" ""
+			(at 469.9 251.46 0)
+			(effects
+				(font
+					(size 1.27 1.27)
+				)
+				(hide yes)
+			)
+		)
+		(property "Description" ""
+			(at 469.9 251.46 0)
+			(effects
+				(font
+					(size 1.27 1.27)
+				)
+				(hide yes)
+			)
+		)
+		(pin "1"
+		)
+		(instances
+			(project "interfejs_digi"
+				(path "/7f52d787-caa3-4a92-b1b2-19d554dc29a4"
+					(reference "#PWR040")
+					(unit 1)
+				)

Commit message: zmiana wyjscia starujacego
Parts:
- added Q4, Q5, Q6: 2N7002, Package_TO_SOT_SMD:SOT-23, symbol Transistor_FET:2N7002
- added R19, R20, R21: 22k, Resistor_SMD:R_0603_1608Metric, symbol Device:R_Small
Connections:
- net +5V: now also R10.2, R11.2, R12.1, R16.1, R17.1, R18.1, R7.2, R8.2, R19.1, R20.1, R21.1; no longer D6.2 (A)
- net CAT1_RX_TTL: now also D8.1 (K); no longer D8.2 (A)
- net CAT1_TX_TTL: now also D10.1 (K); no longer D10.2 (A)
- net CAT2_RX_TTL: now also D7.1 (K); no longer D7.2 (A)
- net CAT2_TX_TTL: now also D9.1 (K); no longer D9.2 (A)
- net CW: now also D3.1 (K), Q6.1 (G); no longer Q3.1 (G), R11.2
- net CW_OUT: now also RJ1.6
- net FSK: now also D2.1 (K); no longer R8.2
- net FSK_OUT: now also Q4.3 (D); no longer Q2.3 (D)
- net GND: now also D6.1 (K), Q4.2 (S), Q5.2 (S), Q6.2 (S); no longer D1.1 (K), D2.1 (K), D3.1 (K), R10.1, R12.1, R16.1, R17.1, R18.1, RJ1.6
- net PTT: now also D1.1 (K), Q5.1 (G); no longer Q1.1 (G), R7.2
- net at R12.2: now also D7.2 (A); no longer D7.1 (K)
- net at R17.2: now also D9.2 (A); no longer D9.1 (K)
- net at R18.2: now also D10.2 (A); no longer D10.1 (K)
- net at R16.2: now also D8.2 (A); no longer D8.1 (K)
- new net: Q1.1 (G), Q5.3 (D), R20.2
- new net: Q3.1 (G), Q6.3 (D), R21.2
- new net: Q2.3 (D), Q4.1 (G), R19.2
- new net: D6.2 (A), R10.1
Other:
- moved on the sheet: D1, D10, D2, D3, D6, D7, D8, D9, Q2, R10, R11, R12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

Commit message: update
Parts:
- U7: DESCRIPTION CP2105 Dual USB 2.0 to UART (RS485) Bridge Interface Evalua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 -> (none)
Other:
- moved on the sheet: C1, C10, C11, C12, C13, C14, C15, C16, C17, C18, C19, C2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
